Commit message: simulate a VLP 16 on the ground robot

File: src/mybot_description/urdf/mybot.xacro (robot description, xacro)
@@ -3,4 +3,6 @@
   <xacro:property name="cameraSize" value="0.05"/>
   <xacro:property name="cameraMass" value="0.1"/>
+  <xacro:arg name="gpu" default="false"/>
+  <xacro:property name="gpu" value="$(arg gpu)" />
   <xacro:include filename="$(find mybot_description)/urdf/mybot.gazebo" />
   <xacro:include filename="$(find mybot_description)/urdf/materials.xacro" />
@@ -190,3 +192,7 @@
     </inertial>
   </link>
+  <xacro:include filename="$(find lidar_description)/urdf/VLP-16.urdf.xacro"/>
+ <xacro:VLP-16 parent="chassis" name="velodyne" topic="/velodyne_points" hz="10" samples="440" gpu="${gpu}">
+    <origin xyz="0 0 0.05" rpy="0 0 0" />
+  </xacro:VLP-16>
 </robot>

Commit message: IMU sensor

File: src/mybot_description/urdf/mybot.xacro (robot description, xacro)
@@ -3,4 +3,6 @@
   <xacro:property name="cameraSize" value="0.05"/>
   <xacro:property name="cameraMass" value="0.1"/>
+  <xacro:property name="imuSize" value="0.04"/>
+  <xacro:property name="imuMass" value="0.1"/>
   <xacro:arg name="gpu" default="false"/>
   <xacro:property name="gpu" value="$(arg gpu)" />
@@ -192,7 +194,34 @@
     </inertial>
   </link>
+  <joint name="imu_joint" type="fixed">
+    <axis xyz="1 0 0"/>
+    <origin xyz="0.0 0.0 0.06" rpy="0 0 0"/>
+    <parent link="chassis"/>
+    <child link="imu_link"/>
+  </joint>
+  <link name="imu_link">
+    <inertial>
+      <mass value="${imuMass}"/>
+      <origin rpy="0 0 0" xyz="0 0 0"/>
+      <box_inertia m="${imuMass}" x="${imuSize}" y="${imuSize}" z="${imuSize}" />
+      <inertia ixx="1e-6" ixy="0" ixz="0" iyy="1e-6" iyz="0" izz="1e-6" />
+    </inertial>
+    <visual>
+      <origin rpy="0 0 0" xyz="0 0 0"/>
+      <geometry>
+        <box size="${imuSize} ${imuSize} ${imuSize}"/>
+      </geometry>
+      <material name="red"/>
+    </visual>
+    <collision>
+      <origin rpy="0 0 0" xyz="0 0 0"/>
+      <geometry>
+        <box size="${imuSize} ${imuSize} ${imuSize}"/>
+      </geometry>
+    </collision>
+  </link>
   <xacro:include filename="$(find lidar_description)/urdf/VLP-16.urdf.xacro"/>
- <xacro:VLP-16 parent="chassis" name="velodyne" topic="/velodyne_points" hz="10" samples="440" gpu="${gpu}">
-    <origin xyz="0 0 0.05" rpy="0 0 0" />
+  <xacro:VLP-16 parent="chassis" name="velodyne" topic="/velodyne_points" hz="10" samples="440" gpu="${gpu}">
+    <origin xyz="-0.1 0 0.06" rpy="0 0 0" />
   </xacro:VLP-16>
 </robot>
